File: 2060-ORIO2.sch (KiCad schematic (older format))
At the start: 160 parts, among them J1 TBL001-500-02GY-2GY, J101 RaspberryPI-B+header, J133 Conn_02x05_Odd_Even, J134 Conn_01x04, J301 Conn_01x08, J302 Conn_01x08, J303 Conn_01x08, J304 Conn_01x08, J305 Conn_01x08, J306 Conn_01x08, J307 Conn_01x08, J308 Conn_01x08, J321 Conn_01x08, J322 Conn_01x08, J323 Conn_01x08, J331 Conn_01x08, J332 Conn_01x08, J333 Conn_01x08, J341 Conn_01x10, J342 Conn_01x10, J343 Conn_01x10, J35 Conn_01x02, J351 Conn_01x10, J352 Conn_01x10, J353 Conn_01x10, J354 Conn_01x10, Q101 DMG2305UX-13, Q102 ULN2803ADWR, Q103 DMMT5401, SW101 SW_DIP_x08, U1 TPS563231, U10 SN74LVC4245AN, U102 AZ1117CH-3.3TRG1, U103 AZ1117CH-1.2, U104 ICE40HX4K-TQ144, U105 MCP3008, U11 AZ1117CH-3.3TRG1, U12 AP3012, U2 TPS563231, U3 SN74LVC4245AN, U4 SN74LVC4245AN, U5 SN74LVC4245AN, U6 SN74LVC4245AN, U7 SN74LVC4245AN, U8 TPS563231, U9 SN74LVC4245AN, Y101 XLH536025_000000I

Commit message: checkpoint
Parts:
- removed J133: Conn_02x05_Odd_Even, Connector_PinHeader_2.54mm:PinHeader_2x05_P2.54mm_Vertical, symbol Connector_Generic:Conn_02x05_Odd_Even
- removed J321: Conn_01x08, Connector_PinHeader_2.54mm:PinHeader_1x08_P2.54mm_Vertical, symbol Connector_Generic:Conn_01x08
- removed J341, J342, J343: Conn_01x10, Connector_PinHeader_2.54mm:PinHeader_1x10_P2.54mm_Vertical, symbol Connector_Generic:Conn_01x10
- removed Q101: DMG2305UX-13, digikey-footprints:SOT-23-3, symbol dk_Transistors-FETs-MOSFETs-Single:DMG2305UX-13
- removed Q103: DMMT5401, Package_TO_SOT_SMD:SOT-23-6, symbol 2060-ORIO2-rescue:DMMT5401-JWlib
- removed R101, R102: 22, Resistor_SMD:R_0603_1608Metric_Pad1.05x0.95mm_HandSolder, symbol Device:R
- removed RN102, RN103: R_Pack08, Resistor_SMD:R_Array_Convex_8x0602, symbol Device:R_Pack08
- added C3, C39, C40, C41, C42, C43, C44, C45: X, Capacitor_SMD:C_0603_1608Metric_Pad1.05x0.95mm_HandSolder, symbol Device:C
- added J321: Conn_01x09, Connector_PinHeader_2.54mm:PinHeader_1x09_P2.54mm_Vertical, symbol Connector_Generic:Conn_01x09
- added J341, J342, J343: Conn_01x16, Connector_PinHeader_2.54mm:PinHeader_1x16_P2.54mm_Vertical, symbol Connector_Generic:Conn_01x16
- added R10, R11, R12, R13, R14, R15, R16, R17, R18, R19, R20, R21, R22, R23, R24, R25, R26, R27, R28, R29, R30, R31, R9: X, Resistor_SMD:R_0603_1608Metric_Pad1.05x0.95mm_HandSolder, symbol Device:R
- U12: footprint Package_TO_SOT_SMD:SOT-23-5_HandSoldering -> Package_TO_SOT_SMD:SOT-23-5
Connections:
- net labels added: ADC_CLK, ADC_SI, ADC_SO, FIO0, FIO1, FIO10, FIO11, FIO12, FIO13, FIO14, FIO15, FIO2, FIO3, FIO4, FIO5, FIO6, FIO7, FIO8, FIO9, FPGA_CE0, FPGA_DIN0, FPGA_DIN1, FPGA_DIN2, FPGA_DIN3, FPGA_DIN4, FPGA_DIN5, FPGA_DIN6, FPGA_DIN7, FPGA_DOUT0, FPGA_DOUT1, FPGA_DOUT2, FPGA_DOUT3, FPGA_DOUT4, FPGA_DOUT5, FPGA_DOUT6, FPGA_DOUT7, FPGA_PWM10, FPGA_PWM11, FPGA_PWM12, FPGA_PWM13, FPGA_PWM14, FPGA_PWM15, FPGA_QA0, FPGA_QA1, FPGA_QA2, FPGA_QA3, FPGA_QA4, FPGA_QA5, FPGA_QA6, FPGA_QA7, FPGA_QA8, FPGA_QA9, FPGA_QB0, FPGA_QB1, FPGA_QB2, FPGA_QB3, FPGA_QB4, FPGA_QB5, FPGA_QB6, FPGA_QB7, FPGA_QB8, FPGA_QB9, FPGA_SCK, FPGA_SDI, FPGA_SDO, FPGA_SS, GPIO16, GPIO23, GPIO24, PB0, PB1, PWM10, PWM11, PWM12, PWM13, PWM14, PWM15, QA3, SPI_MISO, SPI_MOSI, SPI_SCLK, VBATT_DIV, ~ADC_CS
- net labels removed: ADC0_11, FC3_MISO, FC3_MOSI, FC3_SCK, FC3_SSEL0, FC3_SSEL1, FC3_SSEL2, FC3_SSEL3, FPGA_MISO, FPGA_MOSI, FPGA_SCLK, FPGA_SSEL, IOB_102, IOB_103, IOB_104, IOB_82, IOB_91, IOB_94, IOB_95, IOB_96, IOL_10A, IOL_10B, IOL_12A, IOL_12B, IOL_13A, IOL_13B, IOL_14A, IOL_14B, IOL_17A, IOL_17B, IOL_2A, IOL_2B, IOL_3A, IOL_3B, IOL_4A, IOL_4B, IOL_5A, IOL_5B, IOL_8A, IOL_8B, IOR_109, IOR_110, IOR_111, IOR_112, IOR_114, IOR_115, IOR_116, IOR_117, IOR_118, IOR_119, IOR_120, IOR_128, IOR_136, IOR_137, IOR_138, IOR_139, IOR_140, IOR_141, IOR_144, IOR_146, IOR_147, IOR_148, IOR_152, IOR_160, IOR_161, IOR_164, IOR_165, IOR_166, IOR_167, IOT_168, IOT_169, IOT_170, IOT_171, IOT_172, IOT_173, IOT_174, IOT_177, IOT_178, IOT_179, IOT_181, IOT_190, IOT_191, IOT_192, IOT_197, IOT_198, IOT_206, IOT_212, IOT_213, IOT_214, IOT_215, IOT_216, IOT_217, IOT_219, IOT_220, IOT_221, IOT_222, Qa3
- wire segments 932 -> 1056
- no-connect marks 4 -> 34
Other:
- note added: "I2C (Breakout of the PI I2C pins w/3.3v power & pull ups)"
- note added: "PWM w/output level shifter"
- note added: "Shunt J35 for 5V.\nRemove for 3.3V."
- note removed: "I2C (Breakout of the PI I2C pins w/3.3v pull up)"
- note removed: "PI Hat Ideal Diode"
- note removed: "PWM"
- note removed: "PWM output level shifter"
- note removed: "SPI (Breakout of the PI SPI pins)\nShared with the FPGA."
- note removed: "Shunt J35 for 3.3V.\nRemove for 5V."
- moved on the sheet: C21, C22, C23, C24, C25, C26, C27, C28, C29, C30, C31, C32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

Commit message: Dev checkpoint (first version passing DRC)
Parts:
- D8: value 1N5819 -> DB2460600L; footprint (none) -> Diode_SMD:D_SOD-128
- L3: footprint Inductor_SMD:L_Bourns_SRN6045TA -> Inductor_SMD:L_Taiyo-Yuden_NR-40xx_HandSoldering
- U1, U2, U8: footprint Package_TO_SOT_SMD:SOT-563 -> jb-footprint:SOT-563
Connections:
- net PI_5 is gone; now on net 5V_PI: J101.2 (5V), J101.4 (5V)
Other:
- moved on the sheet: C2, D8, R7, R8
Changed lines of the file:
@@
 	1    0    0    -1
 $EndComp
-Text Label 17150 1250 2    50   ~ 0
-PI_5
 Text Label 13800 2150 0    50   ~ 0
 FPGA_SDI
@@
 F 0 "U1" H 2400 12117 50  0000 C CNN
 F 1 "TPS563231" H 2400 12026 50  0000 C CNN
-F 2 "Package_TO_SOT_SMD:SOT-563" H 2450 11500 50  0001 L CNN
+F 2 "jb-footprint:SOT-563" H 2450 11500 50  0001 L CNN
 F 3 "" H 2400 11750 50  0001 C CNN
 	1    2400 11750
@@
 F 0 "U2" H 2450 14067 50  0000 C CNN
 F 1 "TPS563231" H 2450 13976 50  0000 C CNN
-F 2 "Package_TO_SOT_SMD:SOT-563" H 2500 13450 50  0001 L CNN
+F 2 "jb-footprint:SOT-563" H 2500 13450 50  0001 L CNN
 F 3 "" H 2450 13700 50  0001 C CNN
 	1    2450 13700
@@
 F 0 "U8" H 2350 9767 50  0000 C CNN
 F 1 "TPS563231" H 2350 9676 50  0000 C CNN
-F 2 "Package_TO_SOT_SMD:SOT-563" H 2400 9150 50  0001 L CNN
+F 2 "jb-footprint:SOT-563" H 2400 9150 50  0001 L CNN
 F 3 "" H 2350 9400 50  0001 C CNN
 	1    2350 9400
@@
 F 0 "L3" V 7300 14700 50  0000 C CNN
 F 1 "10uH" V 7200 14650 50  0000 C CNN
-F 2 "Inductor_SMD:L_Bourns_SRN6045TA" H 7100 14650 50  0001 C CNN
+F 2 "Inductor_SMD:L_Taiyo-Yuden_NR-40xx_HandSoldering" H 7100 14650 50  0001 C CNN
 F 3 "~" H 7100 14650 50  0001 C CNN
 F 4 "" V 7200 14450 50  0001 C CNN "Digi-Key_PN"
@@
 	7250 14650 7600 14650
 Wire Wire Line
-	7600 14650 7600 14950
-Wire Wire Line
-	7600 14950 7400 14950
+	7850 14950 7600 14950
 $Comp
 L Device:D_Schottky_ALT D8
 U 1 1 6DA29F88
-P 7750 14950
-F 0 "D8" H 7750 14733 50  0000 C CNN
-F 1 "1N5819" H 7750 14824 50  0000 C CNN
-F 2 "" H 7750 14950 50  0001 C CNN
-F 3 "~" H 7750 14950 50  0001 C CNN
-	1    7750 14950
+P 8000 14950
+F 0 "D8" H 8000 14700 50  0000 C CNN
+F 1 "DB2460600L" H 8000 14800 50  0000 C CNN
+F 2 "Diode_SMD:D_SOD-128" H 8000 14950 50  0001 C CNN
+F 3 "~" H 8000 14950 50  0001 C CNN
+	1    8000 14950
 	-1   0    0    1
 $EndComp
-Connection ~ 7600 14950
 $Comp
 L Device:R R?
 U 1 1 6DE228ED
-P 8150 15500
+P 8400 15500
 AR Path="/5BBE5CCD/6DE228ED" Ref="R?"  Part="1"
 AR Path="/6DE228ED" Ref="R8"  Part="1"
 AR Path="/5CF9559A/6DE228ED" Ref="R?"  Part="1"
 AR Path="/5ECC13DB/6DE228ED" Ref="R?"  Part="1"
-F 0 "R8" V 8050 15500 50  0000 C CNN
-F 1 "5K1" V 8150 15500 50  0000 C CNN
-F 2 "Resistor_SMD:R_0603_1608Metric_Pad1.05x0.95mm_HandSolder" V 8080 15500 50  0001 C CNN
-F 3 "~" H 8150 15500 50  0001 C CNN
-F 4 "" H 8150 15500 50  0001 C CNN "Digi-Key_PN"
-	1    8150 15500
+F 0 "R8" V 8300 15500 50  0000 C CNN
+F 1 "5K1" V 8400 15500 50  0000 C CNN
+F 2 "Resistor_SMD:R_0603_1608Metric_Pad1.05x0.95mm_HandSolder" V 8330 15500 50  0001 C CNN
+F 3 "~" H 8400 15500 50  0001 C CNN
+F 4 "" H 8400 15500 50  0001 C CNN "Digi-Key_PN"
+	1    8400 15500
 	1    0    0    -1
 $EndComp
@@
 L Device:R R?
 U 1 1 6DE228F4
-P 8150 15100
+P 8400 15100
 AR Path="/5BBE5CCD/6DE228F4" Ref="R?"  Part="1"
 AR Path="/6DE228F4" Ref="R7"  Part="1"
 AR Path="/5CF9559A/6DE228F4" Ref="R?"  Part="1"
 AR Path="/5ECC13DB/6DE228F4" Ref="R?"  Part="1"
-F 0 "R7" V 8050 15100 50  0000 C CNN
-F 1 "92K82" V 8150 15100 50  0000 C CNN
-F 2 "Resistor_SMD:R_0603_1608Metric_Pad1.05x0.95mm_HandSolder" V 8080 15100 50  0001 C CNN
-F 3 "~" H 8150 15100 50  0001 C CNN
-F 4 "" H 8150 15100 50  0001 C CNN "Digi-Key_PN"
-	1    8150 15100
+F 0 "R7" V 8300 15100 50  0000 C CNN
+F 1 "92K82" V 8400 15100 50  0000 C CNN
+F 2 "Resistor_SMD:R_0603_1608Metric_Pad1.05x0.95mm_HandSolder" V 8330 15100 50  0001 C CNN
+F 3 "~" H 8400 15100 50  0001 C CNN
+F 4 "" H 8400 15100 50  0001 C CNN "Digi-Key_PN"
+	1    8400 15100
 	1    0    0    -1
 $EndComp
@@
 L power:GND #PWR0118
 U 1 1 6DE228FC
-P 8150 15750
-F 0 "#PWR0118" H 8150 15500 50  0001 C CNN
-F 1 "GND" H 8155 15577 50  0001 C CNN
-F 2 "" H 8150 15750 50  0001 C CNN
-F 3 "" H 8150 15750 50  0001 C CNN
-	1    8150 15750
+P 8400 15750
+F 0 "#PWR0118" H 8400 15500 50  0001 C CNN
+F 1 "GND" H 8405 15577 50  0001 C CNN
+F 2 "" H 8400 15750 50  0001 C CNN
+F 3 "" H 8400 15750 50  0001 C CNN
+	1    8400 15750
 	1    0    0    -1
 $EndComp
 Wire Wire Line
-	8150 15750 8150 15650
+	8400 15750 8400 15650
 Wire Wire Line
-	7900 14950 8150 14950
-Connection ~ 8150 14950
+	8150 14950 8400 14950
+Connection ~ 8400 14950
 Wire Wire Line
-	8150 14950 8300 14950
+	8400 14950 8550 14950
 Wire Wire Line
-	8150 15250 8150 15300
+	8400 15250 8400 15300
 Wire Wire Line
-	7400 15050 7800 15050
+	7400 15050 8050 15050
 Wire Wire Line
-	7800 15050 7800 15300
+	8050 15050 8050 15300
 Wire Wire Line
-	7800 15300 8150 15300
-Connection ~ 8150 15300
+	8050 15300 8400 15300
+Connection ~ 8400 15300
 Wire Wire Line
-	8150 15300 8150 15350
+	8400 15300 8400 15350
 Wire Wire Line
 	7400 15150 7400 15500
@@
 L Device:C C?
 U 1 1 6E428459
-P 8400 15300
+P 8650 15300
 AR Path="/5F66828B/6E428459" Ref="C?"  Part="1"
 AR Path="/6E428459" Ref="C2"  Part="1"
-F 0 "C2" H 8515 15346 50  0000 L CNN
-F 1 "1uF" H 8515 15255 50  0000 L CNN
-F 2 "Capacitor_SMD:C_0603_1608Metric_Pad1.05x0.95mm_HandSolder" H 8438 15150 50  0001 C CNN
-F 3 "~" H 8400 15300 50  0001 C CNN
-	1    8400 15300
+F 0 "C2" H 8765 15346 50  0000 L CNN
+F 1 "1uF" H 8765 15255 50  0000 L CNN
+F 2 "Capacitor_SMD:C_0603_1608Metric_Pad1.05x0.95mm_HandSolder" H 8688 15150 50  0001 C CNN
+F 3 "~" H 8650 15300 50  0001 C CNN
+	1    8650 15300
 	1    0    0    -1
 $EndComp
 Wire Wire Line
-	8400 15150 8400 14950
-Connection ~ 8400 14950
+	8650 15150 8650 14950
+Connection ~ 8650 14950
 Wire Wire Line
-	8400 14950 8500 14950
+	8650 14950 8750 14950
 Wire Wire Line
-	8400 15450 8400 15750
+	8650 15450 8650 15750
 $Comp
 L power:GND #PWR0127
 U 1 1 6E631BC2
-P 8400 15750
-F 0 "#PWR0127" H 8400 15500 50  0001 C CNN
-F 1 "GND" H 8405 15577 50  0001 C CNN
-F 2 "" H 8400 15750 50  0001 C CNN
-F 3 "" H 8400 15750 50  0001 C CNN
-	1    8400 15750
+P 8650 15750
+F 0 "#PWR0127" H 8650 15500 50  0001 C CNN
+F 1 "GND" H 8655 15577 50  0001 C CNN
+F 2 "" H 8650 15750 50  0001 C CNN
+F 3 "" H 8650 15750 50  0001 C CNN
+	1    8650 15750
 	1    0    0    -1
 $EndComp
-Text GLabel 8500 14950 2    50   Input ~ 0
+Text GLabel 8750 14950 2    50   Input ~ 0
 VCC_SOL
 Wire Wire Line
@@
 L power:PWR_FLAG #FLG?
 U 1 1 5F35165A
-P 8300 14800
+P 8550 14800
 AR Path="/5F51430C/5F35165A" Ref="#FLG?"  Part="1"
 AR Path="/5F35165A" Ref="#FLG0105"  Part="1"
-F 0 "#FLG0105" H 8300 14875 50  0001 C CNN
-F 1 "PWR_FLAG" H 8300 14973 50  0000 C CNN
-F 2 "" H 8300 14800 50  0001 C CNN
-F 3 "~" H 8300 14800 50  0001 C CNN
-	1    8300 14800
+F 0 "#FLG0105" H 8550 14875 50  0001 C CNN
+F 1 "PWR_FLAG" H 8550 14973 50  0000 C CNN
+F 2 "" H 8550 14800 50  0001 C CNN
+F 3 "~" H 8550 14800 50  0001 C CNN
+	1    8550 14800
 	1    0    0    -1
 $EndComp
 Wire Wire Line
-	8300 14800 8300 14950
-Connection ~ 8300 14950
+	8550 14800 8550 14950
+Connection ~ 8550 14950
 Wire Wire Line
-	8300 14950 8400 14950
+	8550 14950 8650 14950
 $Comp
 L power:PWR_FLAG #FLG?
@@
 NoConn ~ 11350 7500
 NoConn ~ 11350 7600
+Text GLabel 17150 1250 2    50   Input ~ 0
+5V_PI
+Wire Wire Line
+	7600 14650 7600 14950
+Connection ~ 7600 14950
+Wire Wire Line
+	7600 14950 7400 14950
 $EndSCHEMATC

Commit message: Part value & BOM cleanup.
Parts:
- C1, C2, C21: Description (none) -> CAP CER 1UF 25V X5R 0603; Digi-Key_PN (none) -> 1276-1102-1-ND; MPN (none) -> CL10A105KA8NNNC; Manufacturer (none) -> Samsung Electro-Mechanics
- C10, C101, C102, C106, C110, C111, C117, C118, C119, C120, C121, C122, C123, C124, C125, C126, C127, C128, C14, C15, C16, C17, C18, C19, C20, C22, C23, C24, C25, C26, C27, C28, C32, C33, C34, C35, C36, C4, C5, C8, C9: Description (none) -> CAP CER 0.1UF 25V X5R 0603; Digi-Key_PN (none) -> 445-6854-1-ND; MPN (none) -> C1608X5R1E104K; Manufacturer (none) -> TDK Corporation
- C103, C104, C107, C108, C37: Description (none) -> CAP CER 10UF 6.3V X5R 0603; Manufacturer (none) -> Samsung Electro-Mechanics
- C105, C109, C38: Description (none) -> CAP CER 22UF 6.3V X5R 0603; Manufacturer (none) -> Samsung Electro-Mechanics
- C11, C29, C6: Description (none) -> CAP CER 10UF 25V X5R 0805; Digi-Key_PN (none) -> 587-2985-1-ND; MPN (none) -> TMK212BBJ106KG-T; Manufacturer (none) -> Taiyo Yuden
- C12, C13, C132, C30, C31, C7: Description (none) -> CAP CER 22UF 10V X5R 0805; Digi-Key_PN (none) -> 490-10746-1-ND; MPN (none) -> GRM21BR61A226ME44L; Manufacturer (none) -> Murata Electronics
- C3, C39, C40, C41, C42, C43, C44, C45: value X -> .1uF; Description (none) -> CAP CER 0.1UF 25V X5R 0603; Digi-Key_PN (none) -> 445-6854-1-ND; MPN (none) -> C1608X5R1E104K; Manufacturer (none) -> TDK Corporation
- D0, D1, D2, D3, D4, D5, D6, D7: Description (none) -> LED GREEN DIFFUSED 0805 SMD; Digi-Key_PN (none) -> 475-1410-1-ND; MPN (none) -> LG R971-KN-1; Manufacturer (none) -> OSRAM Opto Semiconductors Inc.
- D101: Description (none) -> DIODE GEN PURP 800V 10A DO214AB; MPN (none) -> S10KC V7G; Manufacturer (none) -> Taiwan Semiconductor Corporation
- D102: Description (none) -> DIODE GEN PURP 80V 250MA SOD323; Digi-Key_PN (none) -> 1N4448HWS-FDICT-ND; MPN (none) -> 1N4448HWS-7-F; Manufacturer (none) -> Diodes Incorporated
- D8: Description (none) -> DIODE SCHOTTKY 60V 3A TMINIP2; Digi-Key_PN (none) -> DB2460600LCT-ND; MPN (none) -> DB2460600L; Manufacturer (none) -> Panasonic Electronic Components
- J1: Description (none) -> TERMINAL BLOCK, SCREWLESS, 5.00; MPN (none) -> TBL001-500-02GY-2GY; Manufacturer (none) -> CUI Devices
- L1, L102, L2: value 2.2uH -> 4.7uH; Description (none) -> FIXED IND 4.7UH 4.5A 26 MOHM SMD; Digi-Key_PN (none) -> SRN6045TA-4R7MCT-ND; MPN (none) -> SRN6045TA-4R7M; Manufacturer (none) -> Bourns Inc.
- L3: Description (none) -> FIXED IND 10UH 1.3A 85 MOHM SMD; Digi-Key_PN (none) -> 587-2376-1-ND; MPN (none) -> NRG4026T100M; Manufacturer (none) -> Taiyo Yuden
- R1: value K -> 90K; Description (none) -> RES 90.9K OHM 1% 1/10W 0603; Digi-Key_PN (none) -> RMCF0603FT90K9CT-ND; MPN (none) -> RMCF0603FT90K9; Manufacturer (none) -> Stackpole Electronics Inc
- R10, R11, R12, R13, R14, R15, R9: value X -> 33; Description (none) -> RES SMD 33 OHM 1% 1/10W 0603; Digi-Key_PN (none) -> 311-33.0HRCT-ND; MPN (none) -> RC0603FR-0733RL; Manufacturer (none) -> Yageo
- R107: Description (none) -> RES SMD 73.2K OHM 1% 1/10W 0603; Digi-Key_PN (none) -> 311-73.2KHRCT-ND; MPN (none) -> RC0603FR-0773K2L; Manufacturer (none) -> Yageo
- R109, R133, R134, R135, R2, R5: Description (none) -> RES SMD 10K OHM 1% 1/10W 0603; Digi-Key_PN (none) -> 311-10.0KHRCT-ND; MPN (none) -> RC0603FR-0710KL; Manufacturer (none) -> Yageo
- R131, R132: Description (none) -> RES SMD 100 OHM 1% 1/10W 0603; Digi-Key_PN (none) -> 311-100HRCT-ND; MPN (none) -> RC0603FR-07100RL; Manufacturer (none) -> Yageo
- R16, R17, R18, R19, R20, R21, R22, R23, R24, R25, R26, R27, R28, R29, R30, R31: value X -> 4K7; Description (none) -> RES SMD 4.7K OHM 1% 1/10W 0603; Digi-Key_PN (none) -> 311-4.70KHRCT-ND; MPN (none) -> RC0603FR-074K7L; Manufacturer (none) -> Yageo
- R3: value K -> 2K2; Digi-Key_PN (none) -> 311-2.20KHRCT-ND
- R4: value 73K2 -> 45K3; Description (none) -> RES 45.3K OHM 1% 1/10W 0603; Digi-Key_PN (none) -> RMCF0603FT45K3CT-ND; MPN (none) -> RMCF0603FT45K3; Manufacturer (none) -> Stackpole Electronics Inc
- R6: value K -> 16K2; Description (none) -> RES 16.2K OHM 1% 1/10W 0603; Digi-Key_PN (none) -> RMCF0603FT16K2CT-ND; MPN (none) -> RMCF0603FT16K2; Manufacturer (none) -> Stackpole Electronics Inc
- R7: Description (none) -> RES 90.9K OHM 1% 1/10W 0603; Digi-Key_PN (none) -> RMCF0603FT90K9CT-ND; MPN (none) -> RMCF0603FT90K9
- R8: Description (none) -> RES SMD 4.7K OHM 1% 1/10W 0603; Digi-Key_PN (none) -> 311-4.70KHRCT-ND; MPN (none) -> RC0603FR-074K7L; Manufacturer (none) -> Yageo
- RN101, RN104, RN105: value R_Pack08 -> 330; Description (none) -> RES ARRAY 8 RES 330 OHM 1506; Digi-Key_PN (none) -> Y1331CT-ND; MPN (none) -> EXB-2HV331JV; Manufacturer (none) -> Panasonic Electronic Components
- SW101: Description (none) -> SWITCH SLIDE DIP SPST 100MA 20V; MPN (none) -> 210-8MS; Manufacturer (none) -> CTS Electrocomponents
- U1, U2, U8: Description (none) -> Buck, 3A, 17V; Digi-Key_PN (none) -> 296-TPS563231DRLRCT-ND; MPN (none) -> TPS563231DRLR
- U10, U3, U4, U5, U6, U7, U9: Description (none) -> IC TRNSLTR BIDIRECTIONAL 24TSSOP; MPN (none) -> 74LVC4245APW,112; Manufacturer (none) -> Nexperia USA Inc.
- U102, U11: Description (none) -> IC REG LINEAR 3.3V 800MA SOT223; Manufacturer (none) -> Diodes Incorporated
- U103: Description (none) -> IC REG LINEAR 1.2V 800MA SOT223; Manufacturer (none) -> Diodes Incorporated
- U104: Description (none) -> IC FPGA 107 I/O 144TQFP; Manufacturer (none) -> Lattice Semiconductor Corporation
- U105: Description (none) -> IC ADC 10BIT SAR 16SOIC; Digi-Key_PN (none) -> MCP3008-I/SL-ND; MPN (none) -> MCP3008-I/SL; Manufacturer (none) -> Microchip Technology
- U12: Description (none) -> IC REG BOOST ADJ 500MA SOT23-5; Digi-Key_PN (none) -> AP3012KTR-G1DICT-ND; MPN (none) -> AP3012KTR-G1; Manufacturer (none) -> Diodes Incorporated
Other:
- moved on the sheet: J322, J323, RN105

Commit message: Re-annotate schematic, clean silks, add NT1.
Parts:
- added NT1: Net-Tie_2, NetTie:NetTie-2_SMD_Pad0.5mm, symbol Device:Net-Tie_2
- renumbered C101 to C11, C102 to C12, C103 to C13, C106 to C14, C107 to C15, C110 to C16, C111 to C17, C117 to C18, C118 to C19, C119 to C20, C120 to C21, C121 to C22, C122 to C23, C123 to C24, C124 to C25, C125 to C26, C126 to C27, C127 to C28, C128 to C29, C15 to C30, C16 to C31, C17 to C32, C18 to C33, C19 to C34, C20 to C35, C21 to C36, C22 to C37, C3 to C38, C27 to C39, C39 to C40, C40 to C41, C41 to C42, C42 to C43, C43 to C44, C44 to C45, C28 to C46, C29 to C47, C30 to C48, C31 to C49, C32 to C50, C45 to C51, C37 to C52, C38 to C53, C104 to C54, C105 to C55, C108 to C56, C109 to C57, C4 to C58, C23 to C59, C24 to C60, C25 to C61, C26 to C62, C5 to C63, C6 to C64, C132 to C65, C7 to C66, C8 to C67, C33 to C68, C34 to C69, C35 to C70, C36 to C71, C9 to C72, C10 to C73, C11 to C74, C12 to C75, C13 to C76, C14 to C77, C1 to C78, C2 to C79, D102 to D11, D0 to D12, D1 to D13, D2 to D14, D3 to D15, D4 to D16, D5 to D17, D6 to D18, D7 to D19, D8 to D20, D101 to D21, H1 to H11, H5 to H12, H2 to H13, H6 to H14, H3 to H15, H7 to H16, H4 to H17, H8 to H18, J101 to J11, J134 to J12, J332 to J13, J333 to J14, J331 to J15, J351 to J16, J352 to J17, J353 to J18, J354 to J19, J321 to J20, J322 to J21, J323 to J22, J301 to J23, J303 to J24, J305 to J25, J307 to J26, J35 to J27, J341 to J28, J342 to J29, J343 to J30, J306 to J31, J308 to J32, J302 to J33, J304 to J34, J1 to J35, L2 to L11, L102 to L12, L1 to L13, L3 to L14, LOGO101 to LOGO11, Q102 to Q11, R131 to R11, R15 to R12, R9 to R13, R132 to R14, R10 to R15, R11 to R16, R12 to R17, R13 to R18, R14 to R19, R133 to R20, R134 to R21, R135 to R22, R128 to R23, R129 to R24, R127 to R25, R130 to R26, R3 to R27, R16 to R28, R17 to R29, R18 to R30, R19 to R31, R20 to R32, R21 to R33, R22 to R34, R23 to R35, R4 to R36, R5 to R37, R6 to R38, R24 to R39, R25 to R40, R26 to R41, R27 to R42, R28 to R43, R29 to R44, R30 to R45, R31 to R46, R107 to R47, R109 to R48, R1 to R49, R2 to R50, R7 to R51, R8 to R52, RN101 to RN11, RN105 to RN12, RN104 to RN13, S101 to S11, S102 to S12, SW101 to SW11, U104 to U11, U3 to U12, U4 to U13, U5 to U14, U8 to U15, U105 to U16, U11 to U17, U102 to U18, U103 to U19, U1 to U20, U6 to U21, U7 to U22, U9 to U23, U10 to U24, U2 to U25, U12 to U26, Y101 to Y11
Connections:
- net GND: now also NT1.1
- net at U14.3 (A0): now also U14.4 (A1), U14.5 (A2), U14.6 (A3), NT1.2
